Commit message: Swerve Controller Added

File: Anveshika_ws/src/anveshika_description/urdf/anveshika.urdf.xacro (robot description, xacro)
@@ -2,3 +2,4 @@
 <robot name= "anveshika" xmlns:xacro="https://www.ros.org/wiki/xacro">
     <xacro:include filename="rover.xacro"/>
+    <xacro:include filename="ros2_control.xacro" />
 </robot>

File: Anveshika_ws/src/anveshika_description/urdf/rover.xacro (robot description, xacro)
@@ -2,7 +2,7 @@
 <robot xmlns:xacro="https://www.ros.org/wiki/xacro">
     <!-- For RViz -->
-    <!-- <xacro:property name="meshes_address" value="package://anveshika_description/meshes/rover/" /> -->
+    <xacro:property name="meshes_address" value="package://anveshika_description/meshes/rover/" />
     <!-- For Gazebo -->
-    <xacro:property name="meshes_address" value="$(find anveshika_description)/meshes/rover/" />
+    <!-- <xacro:property name="meshes_address" value="$(find anveshika_description)/meshes/rover/" /> -->
     <xacro:property name="inertial_multipier" value="20" />
     <link name="base_footprint"/>
@@ -129,4 +129,11 @@
         <axis xyz="0 0 1"/>
         <limit lower="${-pi/2}" upper="${pi/2}" effort="100" velocity="100" />
+        <command_interface name="position">
+            <param name="min">-${pi/2}</param>
+            <param name="max">${pi/2}</param>
+        </command_interface>
+        <state_interface name="position"/>
+        <state_interface name="velocity"/>
+        <state_interface name="acceleration"/>
     </joint>
     <xacro:motor_mount_link prefix="back_left"
@@ -139,4 +146,11 @@
         <axis xyz="0 0 1"/>
         <limit lower="${-pi/2}" upper="${pi/2}" effort="100" velocity="100" />
+        <command_interface name="position">
+            <param name="min">-${pi/2}</param>
+            <param name="max">${pi/2}</param>
+        </command_interface>
+        <state_interface name="position"/>
+        <state_interface name="velocity"/>
+        <state_interface name="acceleration"/>
     </joint>
     <xacro:motor_mount_link prefix="front_right"
@@ -149,4 +163,11 @@
         <axis xyz="0 0 1"/>
         <limit lower="${-pi/2}" upper="${pi/2}" effort="100" velocity="100" />
+        <command_interface name="position">
+            <param name="min">-${pi/2}</param>
+            <param name="max">${pi/2}</param>
+        </command_interface>
+        <state_interface name="position"/>
+        <state_interface name="velocity"/>
+        <state_interface name="acceleration"/>
     </joint>
     <xacro:motor_mount_link prefix="back_right"
@@ -159,4 +180,11 @@
         <axis xyz="0 0 1"/>
         <limit lower="${-pi/2}" upper="${pi/2}" effort="100" velocity="100" />
+        <command_interface name="position">
+            <param name="min">-${pi/2}</param>
+            <param name="max">${pi/2}</param>
+        </command_interface>
+        <state_interface name="position"/>
+        <state_interface name="velocity"/>
+        <state_interface name="acceleration"/>
     </joint>
     <xacro:macro name="wheel_link" params="prefix x y z r p ya">
@@ -197,4 +225,11 @@
         <origin xyz="0 0.045 -0.006" rpy="0 0 0"/>
         <axis xyz="0 1 0"/>
+        <command_interface name="velocity">
+            <param name="min">-1</param>
+            <param name="max">1</param>
+        </command_interface>
+        <state_interface name="position"/>
+        <state_interface name="velocity"/>
+        <state_interface name="acceleration"/>
     </joint>
     <xacro:wheel_link prefix="back_left"
@@ -206,4 +241,11 @@
         <origin xyz="0 0.045 -0.006" rpy="0 0 0"/>
         <axis xyz="0 1 0"/>
+        <command_interface name="velocity">
+            <param name="min">-1</param>
+            <param name="max">1</param>
+        </command_interface>
+        <state_interface name="position"/>
+        <state_interface name="velocity"/>
+        <state_interface name="acceleration"/>
     </joint>
     <xacro:wheel_link prefix="front_right"
@@ -215,4 +257,11 @@
         <origin xyz="0 -0.045 -0.006" rpy="0 0 0"/>
         <axis xyz="0 1 0"/>
+        <command_interface name="velocity">
+            <param name="min">-1</param>
+            <param name="max">1</param>
+        </command_interface>
+        <state_interface name="position"/>
+        <state_interface name="velocity"/>
+        <state_interface name="acceleration"/>
     </joint>
     <xacro:wheel_link prefix="back_right"
@@ -224,4 +273,11 @@
         <origin xyz="0 -0.045 -0.006" rpy="0 0 0"/>
         <axis xyz="0 1 0"/>
+        <command_interface name="velocity">
+            <param name="min">-1</param>
+            <param name="max">1</param>
+        </command_interface>
+        <state_interface name="position"/>
+        <state_interface name="velocity"/>
+        <state_interface name="acceleration"/>
     </joint>
 </robot>
