Commit message: Added D435i

File: anveshika_description/urdf/anveshika.urdf.xacro (robot description, xacro)
@@ -1,5 +1,5 @@
-<?xml version="1.0"?>
+<?xml version="1.1"?>
 <robot name= "anveshika" xmlns:xacro="https://www.ros.org/wiki/xacro">
-    <xacro:include filename="rover.xacro"/>
-    <xacro:include filename="ros2_control.xacro" />
+    <xacro:include filename="$(find anveshika_description)/urdf/d435i.xacro"/>
+    <xacro:include filename="$(find anveshika_description)/urdf/rover.xacro"/>
 </robot>

File: anveshika_description/urdf/rover.xacro (robot description, xacro)
@@ -1,9 +1,8 @@
-<?xml version="1.0"?>
+<?xml version="1.1"?>
 <robot xmlns:xacro="https://www.ros.org/wiki/xacro">
     <!-- For RViz -->
     <xacro:property name="meshes_address" value="package://anveshika_description/meshes/rover/" />
     <!-- For Gazebo -->
-    <!-- <xacro:property name="meshes_address" value="$(find anveshika_description)/meshes/rover/" /> -->
-    <xacro:property name="inertial_multipier" value="20" />
+    <!-- <xacro:property name="meshes_address" value="$(find anveshika_description)/meshes/rover" /> -->
     <link name="base_footprint"/>
     <joint name="base_joint" type = "fixed">
@@ -15,5 +14,5 @@
         <visual>
             <geometry>
-                <mesh filename="${meshes_address}box.stl"
+                <mesh filename="${meshes_address}/box.stl"
                        scale="0.001 0.001 0.001" />
             </geometry>
@@ -29,13 +28,36 @@
             <origin xyz="0 0 0" rpy="0 0 0"/>
             <mass value="4.0"/>
-            <inertia ixx="${inertial_multipier*0.05835}" ixy = "0" ixz = "${inertial_multipier*-0.0008805}"
-                    iyy="${inertial_multipier*0.06894}" iyz = "0"
-                        izz="${inertial_multipier*0.09218}"/>
+            <inertia ixx="${0.05835}" ixy = "0" ixz = "${-0.0008805}"
+                    iyy="${0.06894}" iyz = "0"
+                        izz="${0.09218}"/>
         </inertial>
     </link>
+    <joint name="realsense_joint" type = "fixed">
+        <parent link="base_link"/>
+        <child link="realsense_d435i_bottom_screw_frame"/>
+        <origin xyz="0.17 0 0.11" rpy="0 0 0"/>
+    </joint>
+    <xacro:sensor_d435i name="realsense_d435i"
+                        topics_ns="camera"
+                        visualize="false"
+                        align_depth="false"
+                        enable_pointCloud="false"
+                        unite_imu_method="false"
+                        accel_fps="250"
+                        gyro_fps="400"
+                        clip_distance="-1.0"
+                        depth_width="1280"
+                        depth_height="720"
+                        depth_fps="30"
+                        infra_width="640"
+                        infra_height="480"
+                        infra_fps="30"
+                        color_width="1920"
+                        color_height="1080"
+                        color_fps="30"/>
     <link name = "left_bogie">
         <visual>
             <geometry>
-                <mesh filename="${meshes_address}left_bogie.stl"
+                <mesh filename="${meshes_address}/left_bogie.stl"
                        scale="0.001 0.001 0.001" />
             </geometry>
@@ -44,5 +66,5 @@
         <collision>
             <geometry>
-                <mesh filename="${meshes_address}collision_bogie.stl"
+                <mesh filename="${meshes_address}/collision_bogie.stl"
                        scale="0.001 0.001 0.001" />
             </geometry>
@@ -52,7 +74,7 @@
             <origin xyz="0 0 0" rpy="0 0 ${pi}"/>
             <mass value="1.0"/>
-            <inertia ixx="${inertial_multipier*0.008645}" ixy = "0" ixz = "${inertial_multipier*0.0001546}"
-                    iyy="${inertial_multipier*0.05017}" iyz = "${inertial_multipier*0.001152}"
-                    izz="${inertial_multipier*0.04221}"/>
+            <inertia ixx="${0.008645}" ixy = "0" ixz = "${0.0001546}"
+                    iyy="${0.05017}" iyz = "${0.001152}"
+                    izz="${0.04221}"/>
         </inertial>
     </link>
@@ -67,5 +89,5 @@
         <visual>
             <geometry>
-                <mesh filename="${meshes_address}right_bogie.stl"
+                <mesh filename="${meshes_address}/right_bogie.stl"
                        scale="0.001 0.001 0.001" />
             </geometry>
@@ -74,5 +96,5 @@
         <collision>
             <geometry>
-                <mesh filename="${meshes_address}collision_bogie.stl"
+                <mesh filename="${meshes_address}/collision_bogie.stl"
                        scale="0.001 0.001 0.001" />
             </geometry>
@@ -82,7 +104,7 @@
             <origin xyz="0 0 0" rpy="0 0 ${pi}"/>
             <mass value="1.0"/>
-            <inertia ixx="${inertial_multipier*0.008645}" ixy = "0" ixz = "${inertial_multipier*0.0001546}"
-                    iyy="${inertial_multipier*0.05017}" iyz = "${inertial_multipier*-0.001152}"
-                    izz="${inertial_multipier*0.04221}"/>
+            <inertia ixx="${0.008645}" ixy = "0" ixz = "${0.0001546}"
+                    iyy="${0.05017}" iyz = "${-0.001152}"
+                    izz="${0.04221}"/>
         </inertial>
     </link>
@@ -99,5 +121,5 @@
             <visual>
                 <geometry>
-                    <mesh filename="${meshes_address}drive_motor_mount.stl"
+                    <mesh filename="${meshes_address}/drive_motor_mount.stl"
                            scale="0.001 0.001 0.001" />
                 </geometry>
@@ -106,5 +128,5 @@
             <collision>
                 <geometry>
-                    <mesh filename="${meshes_address}collision_motor_mount.stl"
+                    <mesh filename="${meshes_address}/collision_motor_mount.stl"
                            scale="0.001 0.001 0.001" />
                 </geometry>
@@ -114,7 +136,7 @@
                 <origin xyz="${x} ${y} ${z}" rpy="${r} ${p} ${ya}"/>
                 <mass value="0.3"/>
-                <inertia ixx="${inertial_multipier*0.0003244}" ixy = "0" ixz = "${inertial_multipier*-0.0002914}"
-                        iyy="${inertial_multipier*0.001012}" iyz = "0"
-                        izz="${inertial_multipier*0.0007519}"/>
+                <inertia ixx="${0.0003244}" ixy = "0" ixz = "${-0.0002914}"
+                        iyy="${0.001012}" iyz = "0"
+                        izz="${0.0007519}"/>
             </inertial>
         </link>
@@ -192,5 +214,5 @@
             <visual>
                 <geometry>
-                    <mesh filename="${meshes_address}wheel.stl"
+                    <mesh filename="${meshes_address}/wheel.stl"
                            scale="0.001 0.001 0.001" />
                 </geometry>
@@ -211,7 +233,7 @@
                 <origin xyz="${x} ${y} ${z}" rpy="${r} ${p} ${ya}"/>
                 <mass value="0.45"/>
-                <inertia ixx="${inertial_multipier*0.001735}" ixy = "0" ixz = "0"
-                        iyy="${inertial_multipier*0.001735}" iyz = "0"
-                        izz="${inertial_multipier*0.0008776}"/>
+                <inertia ixx="${0.001735}" ixy = "0" ixz = "0"
+                        iyy="${0.001735}" iyz = "0"
+                        izz="${0.0008776}"/>
             </inertial>
         </link>

Commit message: Gazebo Spawn Fixed

File: anveshika_description/urdf/anveshika.urdf.xacro (robot description, xacro)
@@ -1,4 +1,4 @@
 <?xml version="1.1"?>
-<robot name= "anveshika" xmlns:xacro="https://www.ros.org/wiki/xacro">
+<robot name="anveshika" xmlns:xacro="https://www.ros.org/wiki/xacro">
     <xacro:include filename="$(find anveshika_description)/urdf/d435i.xacro"/>
     <xacro:include filename="$(find anveshika_description)/urdf/rover.xacro"/>

File: anveshika_description/urdf/rover.xacro (robot description, xacro)
@@ -2,7 +2,5 @@
 <robot xmlns:xacro="https://www.ros.org/wiki/xacro">
     <!-- For RViz -->
-    <xacro:property name="meshes_address" value="package://anveshika_description/meshes/rover/" />
-    <!-- For Gazebo -->
-    <!-- <xacro:property name="meshes_address" value="$(find anveshika_description)/meshes/rover" /> -->
+    <xacro:property name="meshes_address" value="package://anveshika_description/meshes/rover" />
     <link name="base_footprint"/>
     <joint name="base_joint" type = "fixed">
