Commit message: Fixed Gazebo mimic joint

File: anveshika_description/urdf/anveshika.urdf (robot description, URDF)
Before this commit: robot anveshika, 26 links, 25 joints
Joints:
- joint base_left_bogie_joint: limit lower=-1.5707963267948966 upper=1.5707963267948966 effort=100 velocity=100 -> lower=-1.5707963267948966 upper=1.5707963267948966 effort=0 velocity=100
- joint base_right_bogie_joint: axis 0 1 0 -> 0 -1.0 0; limit lower=-1.5707963267948966 upper=1.5707963267948966 effort=100 velocity=100 -> lower=-1.5707963267948966 upper=1.5707963267948966 effort=0 velocity=100; mimic joint=base_left_bogie_joint multiplier=-1 -> joint=base_left_bogie_joint multiplier=1

File: anveshika_description/urdf/anveshika.urdf.xacro (robot description, xacro)
@@ -3,3 +3,4 @@
     <xacro:include filename="$(find anveshika_description)/urdf/d435i.xacro"/>
     <xacro:include filename="$(find anveshika_description)/urdf/rover.xacro"/>
+    <xacro:include filename="$(find anveshika_description)/urdf/gazebo.xacro"/>
 </robot>

File: anveshika_description/urdf/rover.xacro (robot description, xacro)
@@ -31,4 +31,13 @@
         </inertial>
     </link>
+    <gazebo reference="base_link">
+        <material>Gazebo/Red</material>
+        <!-- <sensor name="imu_sensor" type="imu">
+            <always_on>1</always_on>
+            <update_rate>1</update_rate>
+            <visualize>true</visualize>
+            <topic>imu</topic>
+        </sensor> -->
+    </gazebo>
     <joint name="realsense_joint" type = "fixed">
         <parent link="base_link"/>
@@ -77,4 +86,7 @@
         </inertial>
     </link>
+    <gazebo reference="left_bogie">
+        <material>Gazebo/Red</material>
+    </gazebo>
     <joint name="base_left_bogie_joint" type="revolute">
         <parent link="base_link"/>
@@ -82,5 +94,5 @@
         <origin xyz="0 0.190 0.06" rpy="0 0 0"/>
         <axis xyz="0 1 0"/>
-        <limit lower="${-pi/2}" upper="${pi/2}" effort="100" velocity="100" />
+        <limit lower="${-pi/2}" upper="${pi/2}" effort="0" velocity="100" />
     </joint>
     <link name = "right_bogie">
@@ -107,11 +119,14 @@
         </inertial>
     </link>
+    <gazebo reference="right_bogie">
+        <material>Gazebo/Red</material>
+    </gazebo>
     <joint name="base_right_bogie_joint" type="revolute">
         <parent link="base_link"/>
         <child link="right_bogie"/>
         <origin xyz="0 -0.190 0.06" rpy="0 0 0"/>
-        <axis xyz="0 1 0"/>
-        <limit lower="${-pi/2}" upper="${pi/2}" effort="100" velocity="100" />
-        <mimic joint="base_left_bogie_joint" multiplier="-1"/>
+        <axis xyz="0 -1.0 0"/>
+        <limit lower="${-pi/2}" upper="${pi/2}" effort="0" velocity="100" />
+        <mimic joint="base_left_bogie_joint" multiplier="1"/>
     </joint>
     <xacro:macro name="motor_mount_link" params="prefix x y z r p ya">
@@ -139,4 +154,7 @@
             </inertial>
         </link>
+        <gazebo reference="${prefix}_motor_mount">
+            <material>Gazebo/Red</material>
+        </gazebo>
     </xacro:macro>
     <xacro:motor_mount_link prefix="front_left"
@@ -236,4 +254,7 @@
             </inertial>
         </link>
+        <gazebo reference="${prefix}_wheel">
+            <material>Gazebo/Red</material>
+        </gazebo>
     </xacro:macro>
     <xacro:wheel_link prefix="front_left"

Commit message: lidar physical shape added, topic added

File: anveshika_description/urdf/anveshika.urdf (robot description, URDF)
Before this commit: robot anveshika, 26 links, 25 joints
Links:
- added link laser_frame, mass 0.3; collision cylinder length=0.05 radius=0.05; visual cylinder length=0.05 radius=0.05
Joints:
- added joint laser_joint: type fixed, parent base_link, child laser_frame, origin xyz=0 0 0.1 rpy=0 0 0

File: anveshika_description/urdf/gazebo.xacro (robot description, xacro)
@@ -1,27 +1,23 @@
 <?xml version="1.1" encoding="UTF-8"?>
 <robot xmlns:xacro="http://www.ros.org/wiki/xacro">
-    <gazebo>
-        <plugin filename="gz-sim-joint-state-publisher-system" name="gz::sim::systems::JointStatePublisher">
-            <update_rate>50</update_rate>
-            <joint_name>base_left_bogie_joint</joint_name>
-            <joint_name>base_right_bogie_joint</joint_name>
-            <joint_name>left_bogie_front_left_motor_mount_joint</joint_name>
-            <joint_name>left_bogie_back_left_motor_mount_joint</joint_name>
-            <joint_name>right_bogie_front_right_motor_mount_joint</joint_name>
-            <joint_name>right_bogie_back_right_motor_mount_joint</joint_name>
-            <joint_name>front_left_wheel_joint</joint_name>
-            <joint_name>back_left_wheel_joint</joint_name>
-            <joint_name>front_right_wheel_joint</joint_name>
-            <joint_name>back_right_wheel_joint</joint_name>
-            <topic>/joint_states</topic>
-        </plugin>
-        <plugin
-            filename="gz-sim-sensors-system"
-            name="gz::sim::systems::Sensors">
-            <render_engine>ogre2</render_engine>
-        </plugin>
-        <plugin filename="gz-sim-imu-system"
-            name="gz::sim::systems::Imu">
-        </plugin>
-    </gazebo>
+  <gazebo>
+    <plugin filename="gz-sim-joint-state-publisher-system" name="gz::sim::systems::JointStatePublisher">
+      <update_rate>50</update_rate>
+      <joint_name>base_left_bogie_joint</joint_name>
+      <joint_name>base_right_bogie_joint</joint_name>
+      <joint_name>left_bogie_front_left_motor_mount_joint</joint_name>
+      <joint_name>left_bogie_back_left_motor_mount_joint</joint_name>
+      <joint_name>right_bogie_front_right_motor_mount_joint</joint_name>
+      <joint_name>right_bogie_back_right_motor_mount_joint</joint_name>
+      <joint_name>front_left_wheel_joint</joint_name>
+      <joint_name>back_left_wheel_joint</joint_name>
+      <joint_name>front_right_wheel_joint</joint_name>
+      <joint_name>back_right_wheel_joint</joint_name>
+      <topic>/joint_states</topic>
+    </plugin>
+    <plugin filename="gz-sim-sensors-system" name="gz::sim::systems::Sensors">
+      <render_engine>ogre2</render_engine>
+    </plugin>
+    <plugin filename="gz-sim-imu-system" name="gz::sim::systems::Imu"/>
+  </gazebo>
 </robot>

File: anveshika_description/urdf/lidar.xacro (robot description, xacro)
@@ -1,10 +1,11 @@
-<!--This file is partially copied from https://github.com/joshnewans/articubot_one/blob/545acac87ae215d80ef6b28abe6097eb7281d9ff/description/lidar.xacro-->
 <?xml version="1.0"?>
 <robot xmlns:xacro="https://www.ros.org/wiki/xacro">
+  <!-- Joint between base_link and lidar frame -->
   <joint name="laser_joint" type="fixed">
     <parent link="base_link"/>
     <child link="laser_frame"/>
-    <origin xyz="0 0 -0.035" rpy="0 0 0"/>
+    <origin xyz="0 0 0.1" rpy="0 0 0"/>
   </joint>
+  <!-- LiDAR physical link -->
   <link name="laser_frame">
     <visual>
@@ -12,37 +13,54 @@
         <cylinder radius="0.05" length="0.05"/>
       </geometry>
-      <origin xyz="0 0 0" rpy="0 0 0"/>
+      <origin xyz="0 0 -0.14" rpy="0 0 0"/>
       <material name="Grey">
         <color rgba="0.6 0.6 0.6 1"/>
       </material>
     </visual>
+    <collision>
+      <geometry>
+        <cylinder radius="0.05" length="0.05"/>
+      </geometry>
+      <origin xyz="0 0 0" rpy="0 0 0"/>
+    </collision>
+    <inertial>
+      <mass value="0.3"/>
+      <inertia ixx="0.001" ixy="0.0" ixz="0.0"
+               iyy="0.001" iyz="0.0"
+               izz="0.001"/>
+    </inertial>
   </link>
   <gazebo reference="laser_frame">
-        <material>Gazebo/Red</material>
-        <sensor name="laser" type="ray">
-            <pose> 0 0 0 0 0 0 </pose>
-            <visualize>true</visualize>
-            <update_rate>10</update_rate>
-            <ray>
-                <scan>
-                    <horizontal>
-                        <samples>360</samples>
-                        <min_angle>-3.14</min_angle>
-                        <max_angle>3.14</max_angle>
-                    </horizontal>
-                </scan>
-                <range>
-                    <min>0.3</min>
-                    <max>12</max>
-                </range>
-            </ray>
-            <plugin name="laser_controller" filename="libgazebo_ros_ray_sensor.so">
-                <ros>
-                    <argument>~/out:=scan</argument>
-                </ros>
-                <output_type>sensor_msgs/LaserScan</output_type>
-                <frame_name>laser_frame</frame_name>
-            </plugin>
-        </sensor>
-    </gazebo>
+    <material>Gazebo/Red</material>
+    <sensor name="laser_sensor" type="ray">
+      <pose>0 0 0 0 0 0</pose>
+      <visualize>true</visualize>
+      <update_rate>10.0</update_rate>
+      <ray>
+        <scan>
+          <horizontal>
+            <samples>360</samples>
+            <resolution>1</resolution>
+            <min_angle>-3.1415</min_angle>
+            <max_angle>3.1415</max_angle>
+          </horizontal>
+        </scan>
+        <range>
+          <min>0.12</min>
+          <max>12.0</max>
+          <resolution>0.005</resolution>
+        </range>
+        <noise>
+          <type>gaussian</type>
+          <mean>0.0</mean>
+          <stddev>0.002</stddev>
+        </noise>
+      </ray>
+      <plugin name="gz::sim::systems::LaserSensorPlugin"
+              filename="gz-sim-laser-sensor-system">
+        <topic>/scan</topic>
+        <frame_name>laser_frame</frame_name>
+      </plugin>
+    </sensor>
+  </gazebo>
 </robot>

Commit message: finally lidar publishing data

File: anveshika_description/urdf/anveshika.urdf (robot description, URDF)
Before this commit: robot anveshika, 27 links, 26 joints
Joints:
- joint laser_joint: origin xyz=0 0 0.1 rpy=0 0 0 -> xyz=0 0 -0.04 rpy=3.14159265 0 0

File: anveshika_description/urdf/lidar.xacro (robot description, xacro)
@@ -1,11 +1,9 @@
 <?xml version="1.0"?>
 <robot xmlns:xacro="https://www.ros.org/wiki/xacro">
-  <!-- Joint between base_link and lidar frame -->
   <joint name="laser_joint" type="fixed">
-    <parent link="base_link"/>
-    <child link="laser_frame"/>
-    <origin xyz="0 0 0.1" rpy="0 0 0"/>
-  </joint>
-  <!-- LiDAR physical link -->
+  <parent link="base_link"/>
+  <child link="laser_frame"/>
+  <origin xyz="0 0 -0.04" rpy="3.14159265 0 0"/>
+</joint>
   <link name="laser_frame">
     <visual>
@@ -13,5 +11,5 @@
         <cylinder radius="0.05" length="0.05"/>
       </geometry>
-      <origin xyz="0 0 -0.14" rpy="0 0 0"/>
+      <origin xyz="0 0 0" rpy="0 0 0"/>
       <material name="Grey">
         <color rgba="0.6 0.6 0.6 1"/>
@@ -26,4 +24,5 @@
     <inertial>
       <mass value="0.3"/>
+      <origin xyz="0 0 0" rpy="0 0 0"/>
       <inertia ixx="0.001" ixy="0.0" ixz="0.0"
                iyy="0.001" iyz="0.0"
@@ -31,36 +30,31 @@
     </inertial>
   </link>
-  <gazebo reference="laser_frame">
-    <material>Gazebo/Red</material>
-    <sensor name="laser_sensor" type="ray">
-      <pose>0 0 0 0 0 0</pose>
-      <visualize>true</visualize>
-      <update_rate>10.0</update_rate>
-      <ray>
-        <scan>
-          <horizontal>
-            <samples>360</samples>
-            <resolution>1</resolution>
-            <min_angle>-3.1415</min_angle>
-            <max_angle>3.1415</max_angle>
-          </horizontal>
-        </scan>
-        <range>
-          <min>0.12</min>
-          <max>12.0</max>
-          <resolution>0.005</resolution>
-        </range>
-        <noise>
-          <type>gaussian</type>
-          <mean>0.0</mean>
-          <stddev>0.002</stddev>
-        </noise>
-      </ray>
-      <plugin name="gz::sim::systems::LaserSensorPlugin"
-              filename="gz-sim-laser-sensor-system">
-        <topic>/scan</topic>
-        <frame_name>laser_frame</frame_name>
-      </plugin>
-    </sensor>
-  </gazebo>
+  <gazebo reference = "laser_frame">
+        <sensor name="laser" type="gpu_lidar">
+            <always_on>1</always_on>
+            <visualize>true</visualize>
+            <pose>0 0 0 0 0 0</pose>
+            <update_rate>50</update_rate>
+            <topic>scan</topic>
+            <gz_frame_id>laser_frame</gz_frame_id>
+            <lidar>
+                <scan>
+                    <horizontal>
+                        <samples>360</samples>
+                        <min_angle>-3.14159265</min_angle>
+                        <max_angle>3.14159265</max_angle>
+                    </horizontal>
+                </scan>
+                <range>
+                    <min>0.3</min>
+                    <max>12</max>
+                </range>
+                <noise>
+                    <type>gaussian</type>
+                    <mean>0.0</mean>
+                    <stddev>0.025</stddev>
+                </noise>
+            </lidar>
+        </sensor>
+    </gazebo>
 </robot>
